File: lna/lna.sch (EAGLE design)
At the start: 14 parts, among them U1 PSA4-5043, U4 MCP5301

Commit message: lna: add pdf schematics
Other:
- note removed: "c0g np0"
Changed lines of the file:
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@@
 <wire x1="177.8" y1="81.28" x2="114.3" y2="81.28" width="0.1524" layer="97"/>
 <text x="116.84" y="119.38" size="5.08" layer="97">LDO</text>
-<text x="35.56" y="35.56" size="1.778" layer="91">c0g np0</text>
 <text x="7.62" y="109.22" size="1.778" layer="97">50Ohm Coplanar Waveguide:
 PCB: 1.6mm 4.2 Et

Commit message: hw: correct lna part number
Parts:
- U4: value MCP5301 -> MIC5301
Changed lines of the file:
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@@
 <part name="C10" library="rcl" deviceset="C-EU" device="C0603" value="1u"/>
 <part name="GND3" library="supply1" deviceset="GND" device=""/>
-<part name="U4" library="SparkFun-PowerIC" deviceset="V_REG_LDO" device="SMD" value="MCP5301"/>
+<part name="U4" library="SparkFun-PowerIC" deviceset="V_REG_LDO" device="SMD" value="MIC5301"/>
 <part name="GND10" library="supply1" deviceset="GND" device=""/>
 <part name="C11" library="rcl" deviceset="C-EU" device="C0603" value=".1u"/>
